Commit message: fix bug_4_13_1

File: eli_cs_robot_description/urdf/cs_macro.xacro (robot description, xacro)
@@ -103,4 +103,5 @@
           <xacro:get_mesh name="base" type="visual"/>
         </geometry>
+        <xacro:get_material name="base" type="visual"/>
       </visual>
       <collision>
@@ -118,4 +119,5 @@
           <xacro:get_mesh name="shoulder" type="visual"/>
         </geometry>
+        <xacro:get_material name="shoulder" type="visual"/>
       </visual>
       <collision>
@@ -133,4 +135,5 @@
           <xacro:get_mesh name="upperarm" type="visual"/>
         </geometry>
+        <xacro:get_material name="upperarm" type="visual"/>
       </visual>
       <collision>
@@ -148,4 +151,5 @@
           <xacro:get_mesh name="forearm" type="visual"/>
         </geometry>
+        <xacro:get_material name="forearm" type="visual"/>
       </visual>
       <collision>
@@ -163,4 +167,5 @@
           <xacro:get_mesh name="wrist_1" type="visual"/>
         </geometry>
+        <xacro:get_material name="wrist_1" type="visual"/>
       </visual>
       <collision>
@@ -178,4 +183,5 @@
           <xacro:get_mesh name="wrist_2" type="visual"/>
         </geometry>
+        <xacro:get_material name="wrist_2" type="visual"/>
       </visual>
       <collision>
@@ -193,4 +199,5 @@
           <xacro:get_mesh name="wrist_3" type="visual"/>
         </geometry>
+        <xacro:get_material name="wrist_3" type="visual"/>
       </visual>
       <collision>

File: eli_cs_robot_description/urdf/inc/cs_common.xacro (robot description, xacro)
@@ -41,4 +41,10 @@
     <xacro:get_mesh_path/>
     <mesh filename="${mesh}"/>
+  </xacro:macro>
+  <xacro:macro name="get_material" params="name type">
+    <xacro:get_visual_params name="${name}" type="${type}"/>
+    <material name="${visual_params['material']['name']}">
+      <color rgba="${visual_params['material']['color']}"/>
+    </material>
   </xacro:macro>
   <xacro:macro name="read_model_data" params="joint_limits_parameters_file kinematics_parameters_file physical_parameters_file visual_parameters_file force_abs_paths">

File: eli_cs_robot_description/urdf_5f/cs.urdf.xacro (robot description, xacro)
@@ -43,5 +43,5 @@
    <xacro:arg name="simulation_controllers" default="" />
    <!-- initial position for simulations (Fake Hardware, Gazebo, Ignition) -->
-   <xacro:arg name="initial_positions_file" default="$(find eli_cs_robot_description)/config/initial_positions.yaml"/>
+   <xacro:arg name="initial_positions_file" default="$(find eli_cs_robot_description)/config/initial_positions_h_type.yaml"/>
    <!-- convert to property to use substitution in function -->
    <xacro:property name="initial_positions_file" default="$(arg initial_positions_file)"/>

File: eli_cs_robot_description/urdf_5f/cs_macro.xacro (robot description, xacro)
@@ -103,4 +103,5 @@
           <xacro:get_mesh name="base" type="visual"/>
         </geometry>
+        <xacro:get_material name="base" type="visual"/>
       </visual>
       <collision>
@@ -118,4 +119,5 @@
           <xacro:get_mesh name="shoulder" type="visual"/>
         </geometry>
+        <xacro:get_material name="shoulder" type="visual"/>
       </visual>
       <collision>
@@ -133,4 +135,5 @@
           <xacro:get_mesh name="upperarm" type="visual"/>
         </geometry>
+        <xacro:get_material name="upperarm" type="visual"/>
       </visual>
       <collision>
@@ -148,4 +151,5 @@
           <xacro:get_mesh name="forearm" type="visual"/>
         </geometry>
+        <xacro:get_material name="forearm" type="visual"/>
       </visual>
       <collision>
@@ -163,4 +167,5 @@
           <xacro:get_mesh name="wrist_1" type="visual"/>
         </geometry>
+        <xacro:get_material name="wrist_1" type="visual"/>
       </visual>
       <collision>
@@ -178,4 +183,5 @@
           <xacro:get_mesh name="wrist_2" type="visual"/>
         </geometry>
+        <xacro:get_material name="wrist_2" type="visual"/>
       </visual>
       <collision>

File: eli_cs_robot_description/urdf_5f/inc/cs_common.xacro (robot description, xacro)
@@ -41,4 +41,10 @@
     <xacro:get_mesh_path/>
     <mesh filename="${mesh}"/>
+  </xacro:macro>
+  <xacro:macro name="get_material" params="name type">
+    <xacro:get_visual_params name="${name}" type="${type}"/>
+    <material name="${visual_params['material']['name']}">
+      <color rgba="${visual_params['material']['color']}"/>
+    </material>
   </xacro:macro>
   <xacro:macro name="read_model_data" params="joint_limits_parameters_file kinematics_parameters_file physical_parameters_file visual_parameters_file force_abs_paths">
